File: _autosave-lipo-discharge-protection-board.kicad_pcb (KiCad board)
At the start: 4 copper layers, 100 x 60 mm, 44 parts, among them J1 XT60, J2 Barrel_Jack, J3 2_PIN_SCREW, J4 Screw_Terminal_01x04, J5 Conn_02x02_Top_Bottom, Q1 AO3400A, Q2 AO3401A, Q3 AO3401A, Q4 AO3401A, Q5 AO3401A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

Commit message: Created pcb design
Other:
- board text added: "!! ONLY SHORT ONE SET OF JUMPERS !!"
- board text added: "CUSTOM CUTOUT VOLTAGE SET"
- board text added: "DC IN"
- board text added: "DC OUT"
- board text added: "GND"
- board text added: "POT"
- board text added: "SVE JE TO RESEARCH AND DEVELOPMENT! - Vesnaa"
- board text added: "V+"
- board text removed: "RV1"
- board text removed: "RV1 FOR CUTOUT VOLTAGE SET"
Changed lines of the file:
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@@
   (general
     (thickness 1.6002)
-    (drawings 11)
+    (drawings 22)
     (tracks 223)
     (zones 0)
@@
     (descr "simple 2-pin terminal block, pitch 5.08mm, revamped version of bornier2")
     (tags "terminal block bornier2")
-    (fp_text reference J3 (at 2.54 -5.08 90) (layer F.SilkS)
+    (fp_text reference J3 (at 3.25 -5 90) (layer F.SilkS)
       (effects (font (size 1 1) (thickness 0.15)))
     )
@@
     (descr "Molex Mini-Fit Jr. Power Connectors, old mpn/engineering number: 5566-04A, example for new mpn: 39-28-x04x, 2 Pins per row, Mounting:  (http://www.molex.com/pdm_docs/sd/039281043_sd.pdf), generated with kicad-footprint-generator")
     (tags "connector Molex Mini-Fit_Jr side entry")
-    (fp_text reference J5 (at 2.1 -3.45 90) (layer F.SilkS)
+    (fp_text reference J5 (at 6.5 -4 90) (layer F.SilkS)
       (effects (font (size 1 1) (thickness 0.15)))
     )
@@
     (tags "capacitor handsolder")
     (attr smd)
-    (fp_text reference R1 (at 0 -1.68 90) (layer F.SilkS)
+    (fp_text reference R1 (at 0 2 90) (layer F.SilkS)
       (effects (font (size 1 1) (thickness 0.15)))
     )
@@
     (tags "capacitor handsolder")
     (attr smd)
-    (fp_text reference R2 (at 0 -1.68 90) (layer F.SilkS)
+    (fp_text reference R2 (at 0 -2 90) (layer F.SilkS)
       (effects (font (size 1 1) (thickness 0.15)))
     )
@@
     (tags "capacitor handsolder")
     (attr smd)
-    (fp_text reference R5 (at 0 -1.68 90) (layer F.SilkS)
+    (fp_text reference R5 (at 0.25 2 90) (layer F.SilkS)
       (effects (font (size 1 1) (thickness 0.15)))
     )
@@
     (tags "capacitor handsolder")
     (attr smd)
-    (fp_text reference R6 (at 0 -1.68 90) (layer F.SilkS)
+    (fp_text reference R6 (at 0 -2 90) (layer F.SilkS)
       (effects (font (size 1 1) (thickness 0.15)))
     )
@@
     (tags "capacitor handsolder")
     (attr smd)
-    (fp_text reference R9 (at 0 -1.68 90) (layer F.SilkS)
+    (fp_text reference R9 (at 0 1.75 90) (layer F.SilkS)
       (effects (font (size 1 1) (thickness 0.15)))
     )
@@
     (tags "capacitor handsolder")
     (attr smd)
-    (fp_text reference R10 (at 0 -1.68 90) (layer F.SilkS)
+    (fp_text reference R10 (at 0 -2 90) (layer F.SilkS)
       (effects (font (size 1 1) (thickness 0.15)))
     )
@@
     (pad 1 np_thru_hole circle (at 0 0) (size 3.2 3.2) (drill 3.2) (layers *.Cu *.Mask))
   )
-  (gr_text "RV1 FOR CUTOUT\nVOLTAGE SET" (at 48 88) (layer F.SilkS)
+  (gr_text V+ (at 9.5 45.5 90) (layer F.SilkS)
+    (effects (font (size 1.524 1.524) (thickness 0.3048)))
+  )
+  (gr_text V+ (at 20.5 61 90) (layer F.SilkS)
+    (effects (font (size 1.524 1.524) (thickness 0.3048)))
+  )
+  (gr_text GND (at 36 61 90) (layer F.SilkS)
+    (effects (font (size 1.524 1.524) (thickness 0.3048)))
+  )
+  (gr_text GND (at 9.5 61 90) (layer F.SilkS)
+    (effects (font (size 1.524 1.524) (thickness 0.3048)))
+  )
+  (gr_text "DC OUT" (at 28 66) (layer F.SilkS)
+    (effects (font (size 1.524 1.524) (thickness 0.3048)))
+  )
+  (gr_text "DC OUT" (at 5 66) (layer F.SilkS)
+    (effects (font (size 1.524 1.524) (thickness 0.3048)))
+  )
+  (gr_text GND (at 26 97 45) (layer F.SilkS)
+    (effects (font (size 1.524 1.524) (thickness 0.3048)))
+  )
+  (gr_text GND (at 9.5 89 90) (layer F.SilkS)
+    (effects (font (size 1.524 1.524) (thickness 0.3048)))
+  )
+  (gr_text "DC IN\n" (at 4 85) (layer F.SilkS)
+    (effects (font (size 1.524 1.524) (thickness 0.3048)))
+  )
+  (gr_text "SVE JE TO RESEARCH \nAND DEVELOPMENT!\n- Vesnaa" (at 59 55) (layer F.SilkS)
+    (effects (font (size 0.8 0.8) (thickness 0.2)) (justify left))
+  )
+  (gr_text "!! ONLY SHORT ONE SET OF JUMPERS !!" (at 56 97) (layer F.SilkS)
+    (effects (font (size 1.524 1.524) (thickness 0.3048)))
+  )
+  (gr_text "CUSTOM CUTOUT\nVOLTAGE SET" (at 48 88) (layer F.SilkS)
     (effects (font (size 1.524 1.524) (thickness 0.3048)) (justify right))
   )
-  (gr_text RV1 (at 76 93.75) (layer F.SilkS)
+  (gr_text POT (at 75.5 93.75) (layer F.SilkS)
     (effects (font (size 1.524 1.524) (thickness 0.3048)))
   )
@@
     (connect_pads (clearance 0.508))
     (min_thickness 0.254)
-    (fill (arc_segments 32) (thermal_gap 0.508) (thermal_bridge_width 0.508) (smoothing fillet) (radius 1))
+    (fill yes (arc_segments 32) (thermal_gap 0.508) (thermal_bridge_width 0.508) (smoothing fillet) (radius 1))
     (polygon
       (pts
@@
     (connect_pads (clearance 0.508))
     (min_thickness 0.254)
-    (fill (arc_segments 32) (thermal_gap 0.508) (thermal_bridge_width 0.508) (smoothing fillet) (radius 1))
+    (fill yes (arc_segments 32) (thermal_gap 0.508) (thermal_bridge_width 0.508) (smoothing fillet) (radius 1))
     (polygon
       (pts
@@
     (connect_pads (clearance 0.508))
     (min_thickness 0.254)
-    (fill (arc_segments 32) (thermal_gap 0.508) (thermal_bridge_width 0.508) (smoothing fillet) (radius 1))
+    (fill yes (arc_segments 32) (thermal_gap 0.508) (thermal_bridge_width 0.508) (smoothing fillet) (radius 1))
     (polygon
       (pts
@@
     (connect_pads (clearance 0.508))
     (min_thickness 0.254)
-    (fill (arc_segments 32) (thermal_gap 0.508) (thermal_bridge_width 0.508) (smoothing fillet) (radius 1))
+    (fill yes (arc_segments 32) (thermal_gap 0.508) (thermal_bridge_width 0.508) (smoothing fillet) (radius 1))
     (polygon
       (pts
