File: _autosave-lipo-discharge-protection-board.kicad_pcb (KiCad board)
At the start: 4 copper layers, 100 x 60 mm, 60 parts, among them J1 XT60, J2 Barrel_Jack, J3 2_PIN_SCREW, J4 Screw_Terminal_01x04, J5 Conn_02x02_Top_Bottom, J6 Conn_01x02_Male, Q1 AO3400A, Q2 AO3400A, Q3 AO3401A, Q4 AO3401A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

Commit message: Added all project files and closing the project
Parts:
- removed the ALARM at (88.8, 92.0)
- added ALARM: LED, LED_THT:LED_D5.0mm, F.Cu at (95.7, 80.4)
- U5: value EL3H7 -> 4N35; footprint lipo-discharge-protection-board:SOIC127P700X210-4N -> Package_DIP:DIP-6_W7.62mm
- moved U5 19.9 mm to (83.6, 92.9), turned to 0 degrees
- moved R22 17.6 mm to (94.7, 77.1), turned to 0 degrees
- moved R23 11.8 mm to (83.0, 89.8), turned to 0 degrees
Connections:
- RV1 pad 3: Net-(RV1-Pad3) -> (no net)
- RV2 pad 3: Net-(RV2-Pad3) -> (no net)
- U5 pad 3: Net-(J6-Pad2) -> (no net)
- U5 pad 4: Net-(J6-Pad1) -> Net-(J6-Pad2)
Routing:
- net Net-(D2-Pad2): track 14.2 -> 38.8 mm
- net Net-(R23-Pad1): track 10.6 -> 4.10 mm
- net Net-(J6-Pad1): track 10.2 -> 12.0 mm
- net Net-(J6-Pad2): track 12.3 -> 13.1 mm
- net Net-(D2-Pad1): track 3.97 -> 3.31 mm
