File: lipo-discharge-protection-board.sch (KiCad schematic (older format))
At the start: 50 parts, among them J1 XT60, J2 2_PIN_SCREW, J3 Barrel_Jack, J4 Screw_Terminal_01x04, J5 Screw_Terminal_01x04, J6 Conn_02x02_Odd_Even, J7 Conn_02x02_Odd_Even, J8 Conn_02x04_Odd_Even, Q1 AO3400A, Q2 AO3401A, Q3 AO3401A, Q4 AO3401A, Q5 AO3401A, U1 XL6009_module, U2 XL6009_module, U3 OPAMP

Commit message: Added LCSC part numbers to components
Parts:
- removed C1, C10, C11, C12, C2, C3, C4, C5, C6, C7, C8, C9: 100n 50V, symbol Device:C
- removed Q3, Q4, Q5: AO3401A, symbol Device:Q_PMOS_GSD
- removed R14, R17, R18, R19: 3k3, symbol Device:R
- added C? (x12): 100n 50V, symbol Device:C
- added Q? (x3): AO3401A, symbol Device:Q_PMOS_GSD
- added R? (x4): 3k3, symbol Device:R
- C13: value 100n -> 100n 50V; LCSC (none) -> C49678
- Q1: LCSC (none) -> C20917
- Q2: LCSC (none) -> AO3401A
- R1: value 0 -> 0R DNF
- R10, R2, R9: value 0R -> 0R DNF
- R11, R8: LCSC (none) -> C17520
- R12: LCSC (none) -> C17414
- R13: LCSC (none) -> C17714
- R15: LCSC (none) -> C17513
- R16: LCSC (none) -> C26010
- R3: LCSC (none) -> C4382
- R4: LCSC (none) -> C27834
- R7: LCSC (none) -> C17673
- U3: LCSC (none) -> C7433

Commit message: Reanotated schematic
Parts:
- gave numbers to parts that had none: 19
Changed lines of the file:
@@
 $EndComp
 $Comp
-L Device:R R?
+L Device:R R18
 U 1 1 61597531
 P 8550 950
-F 0 "R?" H 8620 996 50  0000 L CNN
+F 0 "R18" H 8620 996 50  0000 L CNN
 F 1 "3k3" H 8620 905 50  0000 L CNN
 F 2 "" V 8480 950 50  0001 C CNN
@@
 $EndComp
 $Comp
-L Device:R R?
+L Device:R R17
 U 1 1 61597E64
 P 7950 2350
-F 0 "R?" H 8020 2396 50  0000 L CNN
+F 0 "R17" H 8020 2396 50  0000 L CNN
 F 1 "3k3" H 8020 2305 50  0000 L CNN
 F 2 "" V 7880 2350 50  0001 C CNN
@@
 $EndComp
 $Comp
-L Device:R R?
+L Device:R R19
 U 1 1 61598723
 P 9300 2350
-F 0 "R?" H 9370 2396 50  0000 L CNN
+F 0 "R19" H 9370 2396 50  0000 L CNN
 F 1 "3k3" H 9370 2305 50  0000 L CNN
 F 2 "" V 9230 2350 50  0001 C CNN
@@
 $EndComp
 $Comp
-L Device:R R?
+L Device:R R14
 U 1 1 6159BC57
 P 6700 1750
-F 0 "R?" H 6770 1796 50  0000 L CNN
+F 0 "R14" H 6770 1796 50  0000 L CNN
 F 1 "3k3" H 6770 1705 50  0000 L CNN
 F 2 "" V 6630 1750 50  0001 C CNN
@@
 $EndComp
 $Comp
-L Device:C C?
+L Device:C C8
 U 1 1 615B29CB
 P 2650 5750
-F 0 "C?" H 2765 5796 50  0000 L CNN
+F 0 "C8" H 2765 5796 50  0000 L CNN
 F 1 "100n 50V" H 2765 5705 50  0000 L CNN
 F 2 "" H 2688 5600 50  0001 C CNN
@@
 $EndComp
 $Comp
-L Device:C C?
+L Device:C C7
 U 1 1 615B51D2
 P 2600 7100
-F 0 "C?" H 2715 7146 50  0000 L CNN
+F 0 "C7" H 2715 7146 50  0000 L CNN
 F 1 "100n 50V" H 2715 7055 50  0000 L CNN
 F 2 "" H 2638 6950 50  0001 C CNN
@@
 $EndComp
 $Comp
-L Device:C C?
+L Device:C C2
 U 1 1 615B6251
 P 700 4150
-F 0 "C?" H 815 4196 50  0000 L CNN
+F 0 "C2" H 815 4196 50  0000 L CNN
 F 1 "100n 50V" H 815 4105 50  0000 L CNN
 F 2 "" H 738 4000 50  0001 C CNN
@@
 $EndComp
 $Comp
-L Device:C C?
+L Device:C C10
 U 1 1 615C57A5
 P 3300 5750
-F 0 "C?" H 3415 5796 50  0000 L CNN
+F 0 "C10" H 3415 5796 50  0000 L CNN
 F 1 "100n 50V" H 3415 5705 50  0000 L CNN
 F 2 "" H 3338 5600 50  0001 C CNN
@@
 $EndComp
 $Comp
-L Device:C C?
+L Device:C C12
 U 1 1 615C5C08
 P 3900 5750
-F 0 "C?" H 4015 5796 50  0000 L CNN
+F 0 "C12" H 4015 5796 50  0000 L CNN
 F 1 "100n 50V" H 4015 5705 50  0000 L CNN
 F 2 "" H 3938 5600 50  0001 C CNN
@@
 $EndComp
 $Comp
-L Device:C C?
+L Device:C C9
 U 1 1 615C5EC1
 P 3250 7100
-F 0 "C?" H 3365 7146 50  0000 L CNN
+F 0 "C9" H 3365 7146 50  0000 L CNN
 F 1 "100n 50V" H 3365 7055 50  0000 L CNN
 F 2 "" H 3288 6950 50  0001 C CNN
@@
 $EndComp
 $Comp
-L Device:C C?
+L Device:C C11
 U 1 1 615C6CF2
 P 3850 7100
-F 0 "C?" H 3965 7146 50  0000 L CNN
+F 0 "C11" H 3965 7146 50  0000 L CNN
 F 1 "100n 50V" H 3965 7055 50  0000 L CNN
 F 2 "" H 3888 6950 50  0001 C CNN
@@
 $EndComp
 $Comp
-L Device:C C?
+L Device:C C4
 U 1 1 615C7408
 P 1350 4150
-F 0 "C?" H 1465 4196 50  0000 L CNN
+F 0 "C4" H 1465 4196 50  0000 L CNN
 F 1 "100n 50V" H 1465 4105 50  0000 L CNN
 F 2 "" H 1388 4000 50  0001 C CNN
@@
 $EndComp
 $Comp
-L Device:C C?
+L Device:C C6
 U 1 1 615CA8AB
 P 1950 4150
-F 0 "C?" H 2065 4196 50  0000 L CNN
+F 0 "C6" H 2065 4196 50  0000 L CNN
 F 1 "100n 50V" H 2065 4105 50  0000 L CNN
 F 2 "" H 1988 4000 50  0001 C CNN
@@
 $EndComp
 $Comp
-L Device:C C?
+L Device:C C3
 U 1 1 615CC7DC
 P 1350 2000
-F 0 "C?" H 1465 2046 50  0000 L CNN
+F 0 "C3" H 1465 2046 50  0000 L CNN
 F 1 "100n 50V" H 1465 1955 50  0000 L CNN
 F 2 "" H 1388 1850 50  0001 C CNN
@@
 $EndComp
 $Comp
-L Device:C C?
+L Device:C C5
 U 1 1 615CCE5F
 P 1950 2000
-F 0 "C?" H 2065 2046 50  0000 L CNN
+F 0 "C5" H 2065 2046 50  0000 L CNN
 F 1 "100n 50V" H 2065 1955 50  0000 L CNN
 F 2 "" H 1988 1850 50  0001 C CNN
@@
 $EndComp
 $Comp
-L Device:C C?
+L Device:C C1
 U 1 1 615CD2CE
 P 700 2000
-F 0 "C?" H 815 2046 50  0000 L CNN
+F 0 "C1" H 815 2046 50  0000 L CNN
 F 1 "100n 50V" H 815 1955 50  0000 L CNN
 F 2 "" H 738 1850 50  0001 C CNN
@@
 $EndComp
 $Comp
-L Device:Q_PMOS_GSD Q?
+L Device:Q_PMOS_GSD Q4
 U 1 1 615D36BE
 P 8900 1350
-F 0 "Q?" H 9105 1396 50  0000 L CNN
+F 0 "Q4" H 9105 1396 50  0000 L CNN
 F 1 "AO3401A" H 9105 1305 50  0000 L CNN
 F 2 "" H 9100 1450 50  0001 C CNN
@@
 $EndComp
 $Comp
-L Device:Q_PMOS_GSD Q?
+L Device:Q_PMOS_GSD Q3
 U 1 1 615D4019
 P 8300 2750
-F 0 "Q?" H 8505 2796 50  0000 L CNN
+F 0 "Q3" H 8505 2796 50  0000 L CNN
 F 1 "AO3401A" H 8505 2705 50  0000 L CNN
 F 2 "" H 8500 2850 50  0001 C CNN
@@
 $EndComp
 $Comp
-L Device:Q_PMOS_GSD Q?
+L Device:Q_PMOS_GSD Q5
 U 1 1 615D4DA6
 P 9650 2750
-F 0 "Q?" H 9855 2796 50  0000 L CNN
+F 0 "Q5" H 9855 2796 50  0000 L CNN
 F 1 "AO3401A" H 9855 2705 50  0000 L CNN
 F 2 "" H 9850 2850 50  0001 C CNN

Commit message: Assigned footprints to components
Parts:
- C1, C13, C2, C7, C8, R1, R10, R11, R12, R13, R14, R15, R16, R17, R18, R19, R2, R3, R4, R5, R6, R7, R8, R9: footprint (none) -> Capacitor_SMD:C_0805_2012Metric_Pad1.18x1.45mm_HandSolder
- C10, C11, C12, C3, C4, C5, C6, C9: value 100n 50V -> 10u 50V; footprint (none) -> Capacitor_SMD:C_1206_3216Metric_Pad1.33x1.80mm_HandSolder
- D1: footprint (none) -> Diode_SMD:D_MELF; LCSC (none) -> C8056
- J2: footprint Connector_AMASS:AMASS_XT60-F_1x02_P7.20mm_Vertical -> TerminalBlock:TerminalBlock_bornier-2_P5.08mm
- J3: footprint (none) -> Connector_BarrelJack:BarrelJack_Horizontal
- J4, J5: footprint (none) -> TerminalBlock:TerminalBlock_bornier-4_P5.08mm
- J6, J7: footprint (none) -> Connector_Molex:Molex_Mini-Fit_Jr_5566-04A_2x02_P4.20mm_Vertical
- J8: footprint (none) -> Connector_Molex:Molex_Mini-Fit_Jr_5566-08A_2x04_P4.20mm_Vertical
- Q1, Q2, Q3, Q4, Q5: footprint (none) -> Package_TO_SOT_SMD:SOT-23
- RV1: footprint (none) -> Potentiometer_THT:Potentiometer_Bourns_3296W_Vertical
- U1, U2: footprint (none) -> misc_standard:XL6009_module_SMT
- U3: footprint (none) -> Package_SO:SOIC-8_3.9x4.9mm_P1.27mm
Other:
- moved on the sheet: C13, D1, Q1, Q2, Q3, Q4, Q5, R1, R10, R11, R12, R13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

Commit message: Commit before shrinking to 1ch design
Parts:
- removed J6, J7: Conn_02x02_Odd_Even, Connector_Molex:Molex_Mini-Fit_Jr_5566-04A_2x02_P4.20mm_Vertical, symbol Connector_Generic:Conn_02x02_Odd_Even
- removed J8: Conn_02x04_Odd_Even, Connector_Molex:Molex_Mini-Fit_Jr_5566-08A_2x04_P4.20mm_Vertical, symbol Connector_Generic:Conn_02x04_Odd_Even
- added J6, J7: Conn_02x02_Top_Bottom, Connector_Molex:Molex_Mini-Fit_Jr_5566-04A_2x02_P4.20mm_Vertical, symbol Connector_Generic:Conn_02x02_Top_Bottom
- added J8: Conn_02x04_Top_Bottom, Connector_Molex:Molex_Mini-Fit_Jr_5566-08A_2x04_P4.20mm_Vertical, symbol Connector_Generic:Conn_02x04_Top_Bottom
Other:
- moved on the sheet: C1, C3, C5, J3

Commit message: Created pcb design
Parts:
- removed C11, C9: 10u 50V, Capacitor_SMD:C_1206_3216Metric_Pad1.33x1.80mm_HandSolder, symbol Device:C
- removed C7: 100n 50V, Capacitor_SMD:C_0805_2012Metric_Pad1.18x1.45mm_HandSolder, symbol Device:C
- removed J4: Screw_Terminal_01x04, TerminalBlock:TerminalBlock_bornier-4_P5.08mm, symbol Connector:Screw_Terminal_01x04
- removed J6: Conn_02x02_Top_Bottom, Connector_Molex:Molex_Mini-Fit_Jr_5566-04A_2x02_P4.20mm_Vertical, symbol Connector_Generic:Conn_02x02_Top_Bottom
- removed J8: Conn_02x04_Top_Bottom, Connector_Molex:Molex_Mini-Fit_Jr_5566-08A_2x04_P4.20mm_Vertical, symbol Connector_Generic:Conn_02x04_Top_Bottom
- removed R17, R18, R19: 3k3, Capacitor_SMD:C_0805_2012Metric_Pad1.18x1.45mm_HandSolder, symbol Device:R
- removed U1: XL6009_module, misc_standard:XL6009_module_SMT, symbol xl6009_module:XL6009_module
- added H1, H2, H3, H4: MountingHole, MountingHole:MountingHole_3.2mm_M3, symbol Mechanical:MountingHole
- renumbered C12 to C10, C3 to C2, C2 to C3, C5 to C4, C4 to C5, C8 to C7, C10 to C8, C13 to C9, J3 to J2, J2 to J3, J5 to J4, J7 to J5, U2 to U1, U3 to U2
Connections:
- net +BATT: now also J3.2 (Pin_2); no longer J3.1 (Pin_1)
- net GND: now also J3.1 (Pin_1); no longer J3.2 (Pin_2)
Other:
- moved on the sheet: C1, C10, C2, C3, C4, C5, C6, C7, C8, J1, J2, J3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

Commit message: Updated bad footprints and exported bom
Parts:
- Q2, Q3, Q4, Q5: LCSC AO3401A -> C15127
- R1, R10, R11, R12, R13, R14, R15, R16, R2, R3, R4, R6, R7, R8, R9: footprint Capacitor_SMD:C_0805_2012Metric_Pad1.18x1.45mm_HandSolder -> Resistor_SMD:R_0805_2012Metric_Pad1.20x1.40mm_HandSolder
- R5: value 0 -> 0R; footprint Capacitor_SMD:C_0805_2012Metric_Pad1.18x1.45mm_HandSolder -> Resistor_SMD:R_0805_2012Metric_Pad1.20x1.40mm_HandSolder
- U1: symbol xl6009_module:XL6009_module -> lipo-discharge-protection-board-rescue:XL6009_module-xl6009_module
Changed lines of the file:
@@
 F 0 "R12" H 5470 1296 50  0000 L CNN
 F 1 "10k" H 5470 1205 50  0000 L CNN
-F 2 "Capacitor_SMD:C_0805_2012Metric_Pad1.18x1.45mm_HandSolder" V 5330 1250 50  0001 C CNN
+F 2 "Resistor_SMD:R_0805_2012Metric_Pad1.20x1.40mm_HandSolder" V 5330 1250 50  0001 C CNN
 F 3 "~" H 5400 1250 50  0001 C CNN
 F 4 "C17414" H 5400 1250 50  0001 C CNN "LCSC"
@@
 F 0 "R15" H 6770 2496 50  0000 L CNN
 F 1 "1k" H 6770 2405 50  0000 L CNN
-F 2 "Capacitor_SMD:C_0805_2012Metric_Pad1.18x1.45mm_HandSolder" V 6630 2450 50  0001 C CNN
+F 2 "Resistor_SMD:R_0805_2012Metric_Pad1.20x1.40mm_HandSolder" V 6630 2450 50  0001 C CNN
 F 3 "~" H 6700 2450 50  0001 C CNN
 F 4 "C17513" H 6700 2450 50  0001 C CNN "LCSC"
@@
 F 2 "Package_TO_SOT_SMD:SOT-23" H 7750 1700 50  0001 C CNN
 F 3 "~" H 7550 1600 50  0001 C CNN
-F 4 "AO3401A" H 7550 1600 50  0001 C CNN "LCSC"
+F 4 "C15127" H 7550 1600 50  0001 C CNN "LCSC"
 	1    7550 1600
 	1    0    0    -1
@@
 F 0 "R11" H 4870 2546 50  0000 L CNN
 F 1 "2k2" H 4870 2455 50  0000 L CNN
-F 2 "Capacitor_SMD:C_0805_2012Metric_Pad1.18x1.45mm_HandSolder" V 4730 2500 50  0001 C CNN
+F 2 "Resistor_SMD:R_0805_2012Metric_Pad1.20x1.40mm_HandSolder" V 4730 2500 50  0001 C CNN
 F 3 "~" H 4800 2500 50  0001 C CNN
 F 4 "C17520" H 4800 2500 50  0001 C CNN "LCSC"
@@
 F 0 "R13" H 5920 1246 50  0000 L CNN
 F 1 "47R" H 5920 1155 50  0000 L CNN
-F 2 "Capacitor_SMD:C_0805_2012Metric_Pad1.18x1.45mm_HandSolder" V 5780 1200 50  0001 C CNN
+F 2 "Resistor_SMD:R_0805_2012Metric_Pad1.20x1.40mm_HandSolder" V 5780 1200 50  0001 C CNN
 F 3 "~" H 5850 1200 50  0001 C CNN
 F 4 "C17714" H 5850 1200 50  0001 C CNN "LCSC"
@@
 F 0 "R16" H 7270 1246 50  0000 L CNN
 F 1 "3k3" H 7270 1155 50  0000 L CNN
-F 2 "Capacitor_SMD:C_0805_2012Metric_Pad1.18x1.45mm_HandSolder" V 7130 1200 50  0001 C CNN
+F 2 "Resistor_SMD:R_0805_2012Metric_Pad1.20x1.40mm_HandSolder" V 7130 1200 50  0001 C CNN
 F 3 "~" H 7200 1200 50  0001 C CNN
 F 4 "C26010" H 7200 1200 50  0001 C CNN "LCSC"
@@
 Connection ~ 2300 5050
 $Comp
-L xl6009_module:XL6009_module U1
+L lipo-discharge-protection-board-rescue:XL6009_module-xl6009_module U1
 U 1 1 6152E5F7
 P 4500 4800
@@
 F 0 "R9" V 4143 1050 50  0000 C CNN
 F 1 "0R DNF" V 4234 1050 50  0000 C CNN
-F 2 "Capacitor_SMD:C_0805_2012Metric_Pad1.18x1.45mm_HandSolder" V 4280 1050 50  0001 C CNN
+F 2 "Resistor_SMD:R_0805_2012Metric_Pad1.20x1.40mm_HandSolder" V 4280 1050 50  0001 C CNN
 F 3 "~" H 4350 1050 50  0001 C CNN
 	1    4350 1050
@@
 F 0 "R8" H 4220 2946 50  0000 L CNN
 F 1 "2k2" H 4220 2855 50  0000 L CNN
-F 2 "Capacitor_SMD:C_0805_2012Metric_Pad1.18x1.45mm_HandSolder" V 4080 2900 50  0001 C CNN
+F 2 "Resistor_SMD:R_0805_2012Metric_Pad1.20x1.40mm_HandSolder" V 4080 2900 50  0001 C CNN
 F 3 "~" H 4150 2900 50  0001 C CNN
 F 4 "C17520" H 4150 2900 50  0001 C CNN "LCSC"
@@
 F 0 "R6" V 3800 1600 50  0000 C CNN
 F 1 "0R" V 3900 1600 50  0000 C CNN
-F 2 "Capacitor_SMD:C_0805_2012Metric_Pad1.18x1.45mm_HandSolder" V 3630 1600 50  0001 C CNN
+F 2 "Resistor_SMD:R_0805_2012Metric_Pad1.20x1.40mm_HandSolder" V 3630 1600 50  0001 C CNN
 F 3 "~" H 3700 1600 50  0001 C CNN
 	1    3700 1600
@@
 P 3700 1450
 F 0 "R5" V 3493 1450 50  0000 C CNN
-F 1 "0" V 3584 1450 50  0000 C CNN
-F 2 "Capacitor_SMD:C_0805_2012Metric_Pad1.18x1.45mm_HandSolder" V 3630 1450 50  0001 C CNN
+F 1 "0R" V 3584 1450 50  0000 C CNN
+F 2 "Resistor_SMD:R_0805_2012Metric_Pad1.20x1.40mm_HandSolder" V 3630 1450 50  0001 C CNN
 F 3 "~" H 3700 1450 50  0001 C CNN
 	1    3700 1450
@@
 F 0 "R7" H 4220 1996 50  0000 L CNN
 F 1 "4k7" H 4220 1905 50  0000 L CNN
-F 2 "Capacitor_SMD:C_0805_2012Metric_Pad1.18x1.45mm_HandSolder" V 4080 1950 50  0001 C CNN
+F 2 "Resistor_SMD:R_0805_2012Metric_Pad1.20x1.40mm_HandSolder" V 4080 1950 50  0001 C CNN
 F 3 "~" H 4150 1950 50  0001 C CNN
 F 4 "C17673" H 4150 1950 50  0001 C CNN "LCSC"
@@
 F 0 "R3" H 3620 2396 50  0000 L CNN
 F 1 "5k6" H 3620 2305 50  0000 L CNN
-F 2 "Capacitor_SMD:C_0805_2012Metric_Pad1.18x1.45mm_HandSolder" V 3480 2350 50  0001 C CNN
+F 2 "Resistor_SMD:R_0805_2012Metric_Pad1.20x1.40mm_HandSolder" V 3480 2350 50  0001 C CNN
 F 3 "~" H 3550 2350 50  0001 C CNN
 F 4 "C4382" H 3550 2350 50  0001 C CNN "LCSC"
@@
 F 0 "R1" V 2893 1850 50  0000 C CNN
 F 1 "0R DNF" V 2984 1850 50  0000 C CNN
-F 2 "Capacitor_SMD:C_0805_2012Metric_Pad1.18x1.45mm_HandSolder" V 3030 1850 50  0001 C CNN
+F 2 "Resistor_SMD:R_0805_2012Metric_Pad1.20x1.40mm_HandSolder" V 3030 1850 50  0001 C CNN
 F 3 "~" H 3100 1850 50  0001 C CNN
 	1    3100 1850
@@
 F 0 "R2" V 3215 2000 50  0000 C CNN
 F 1 "0R DNF" V 3306 2000 50  0000 C CNN
-F 2 "Capacitor_SMD:C_0805_2012Metric_Pad1.18x1.45mm_HandSolder" V 3030 2000 50  0001 C CNN
+F 2 "Resistor_SMD:R_0805_2012Metric_Pad1.20x1.40mm_HandSolder" V 3030 2000 50  0001 C CNN
 F 3 "~" H 3100 2000 50  0001 C CNN
 	1    3100 2000
@@
 F 0 "R4" H 3620 3346 50  0000 L CNN
 F 1 "5k1" H 3620 3255 50  0000 L CNN
-F 2 "Capacitor_SMD:C_0805_2012Metric_Pad1.18x1.45mm_HandSolder" V 3480 3300 50  0001 C CNN
+F 2 "Resistor_SMD:R_0805_2012Metric_Pad1.20x1.40mm_HandSolder" V 3480 3300 50  0001 C CNN
 F 3 "~" H 3550 3300 50  0001 C CNN
 F 4 "C27834" H 3550 3300 50  0001 C CNN "LCSC"
@@
 F 0 "R10" V 4450 1200 50  0000 C CNN
 F 1 "0R DNF" V 4550 1200 50  0000 C CNN
-F 2 "Capacitor_SMD:C_0805_2012Metric_Pad1.18x1.45mm_HandSolder" V 4280 1200 50  0001 C CNN
+F 2 "Resistor_SMD:R_0805_2012Metric_Pad1.20x1.40mm_HandSolder" V 4280 1200 50  0001 C CNN
 F 3 "~" H 4350 1200 50  0001 C CNN
 	1    4350 1200
@@
 F 0 "R14" H 6770 2046 50  0000 L CNN
 F 1 "3k3" H 6770 1955 50  0000 L CNN
-F 2 "Capacitor_SMD:C_0805_2012Metric_Pad1.18x1.45mm_HandSolder" V 6630 2000 50  0001 C CNN
+F 2 "Resistor_SMD:R_0805_2012Metric_Pad1.20x1.40mm_HandSolder" V 6630 2000 50  0001 C CNN
 F 3 "~" H 6700 2000 50  0001 C CNN
 F 4 "C26010" H 6700 2000 50  0001 C CNN "LCSC"
@@
 F 2 "Package_TO_SOT_SMD:SOT-23" H 9100 1700 50  0001 C CNN
 F 3 "~" H 8900 1600 50  0001 C CNN
-F 4 "AO3401A" H 8900 1600 50  0001 C CNN "LCSC"
+F 4 "C15127" H 8900 1600 50  0001 C CNN "LCSC"
 	1    8900 1600
 	1    0    0    -1
@@
 F 2 "Package_TO_SOT_SMD:SOT-23" H 8500 3100 50  0001 C CNN
 F 3 "~" H 8300 3000 50  0001 C CNN
-F 4 "AO3401A" H 8300 3000 50  0001 C CNN "LCSC"
+F 4 "C15127" H 8300 3000 50  0001 C CNN "LCSC"
 	1    8300 3000
 	1    0    0    -1
@@
 F 2 "Package_TO_SOT_SMD:SOT-23" H 9850 3100 50  0001 C CNN
 F 3 "~" H 9650 3000 50  0001 C CNN
-F 4 "AO3401A" H 9650 3000 50  0001 C CNN "LCSC"
+F 4 "C15127" H 9650 3000 50  0001 C CNN "LCSC"
 	1    9650 3000
 	1    0    0    -1
