File: lipo-discharge-protection-board.sch (KiCad schematic (older format))
At the start: 44 parts, among them J1 XT60, J2 Barrel_Jack, J3 2_PIN_SCREW, J4 Screw_Terminal_01x04, J5 Conn_02x02_Top_Bottom, Q1 AO3400A, Q2 AO3401A, Q3 AO3401A, Q4 AO3401A, Q5 AO3401A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

Commit message: Updated
Parts:
- added C?: 100n 50V, Capacitor_SMD:C_0805_2012Metric_Pad1.18x1.45mm_HandSolder, symbol Device:C
- added R?: 47R, Capacitor_SMD:C_0805_2012Metric_Pad1.18x1.45mm_HandSolder, symbol Device:R
- added R?: 2k2, Capacitor_SMD:C_0805_2012Metric_Pad1.18x1.45mm_HandSolder, symbol Device:R
- added RV?: 10k, Potentiometer_THT:Potentiometer_Bourns_3296W_Vertical, symbol Device:R_POT
- added U?: OPAMP, Package_SO:SOIC-8_3.9x4.9mm_P1.27mm, symbol pspice:OPAMP
Connections:
- net +BATT: now also RV?.1
- net +VDC: now also R?.1
- net GND: now also C?.1, R?.2, U?.5 (V-)
- net at D1.1 (K), R12.2, U2.2 (-): now also U?.2 (-)
- new net: R?.1, RV?.2, U?.1 (+)
- new net: C?.2, R?.2, U?.4 (V+)
Other:
- moved on the sheet: C10, C3, C5, C6, C7, C8, H1, H2, H3, H4, J4, J5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
